File: GACSA EZ-48.kicad_pcb (KiCad board)
At the start: 2 copper layers, 333.7 x 176.5 mm, 0 parts

Commit message: Project restarted in a modular way
Project restarted in a modular way
Other:
- board outline removed
Changed lines of the file:
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@@
 		(legacy_teardrops no)
 	)
-	(paper "A3")
+	(paper "A4")
 	(layers
 		(0 "F.Cu" signal)
@@
 	)
 	(net 0 "")
-	(gr_line
-		(start 377.307553 49.004446)
-		(end 377.303553 224.496446)
-		(stroke
-			(width 0.05)
-			(type solid)
-		)
-		(layer "Edge.Cuts")
-	)
-	(gr_arc
-		(start 43.603553 49.003553)
-		(mid 43.75 48.65)
-		(end 44.103553 48.503553)
-		(stroke
-			(width 0.05)
-			(type solid)
-		)
-		(layer "Edge.Cuts")
-	)
-	(gr_arc
-		(start 376.803553 48.503552)
-		(mid 377.157106 48.649999)
-		(end 377.303553 49.003552)
-		(stroke
-			(width 0.05)
-			(type solid)
-		)
-		(layer "Edge.Cuts")
-	)
-	(gr_arc
-		(start 44.103553 224.996447)
-		(mid 43.75 224.85)
-		(end 43.603553 224.496447)
-		(stroke
-			(width 0.05)
-			(type solid)
-		)
-		(layer "Edge.Cuts")
-	)
-	(gr_line
-		(start 44.1036 48.503553)
-		(end 376.8036 48.503553)
-		(stroke
-			(width 0.05)
-			(type solid)
-		)
-		(layer "Edge.Cuts")
-	)
-	(gr_line
-		(start 43.599553 224.495553)
-		(end 43.603553 49.003553)
-		(stroke
-			(width 0.05)
-			(type solid)
-		)
-		(layer "Edge.Cuts")
-	)
-	(gr_line
-		(start 44.103553 224.996446)
-		(end 376.803553 224.996446)
-		(stroke
-			(width 0.05)
-			(type solid)
-		)
-		(layer "Edge.Cuts")
-	)
-	(gr_arc
-		(start 377.303553 224.496446)
-		(mid 377.157106 224.849999)
-		(end 376.803553 224.996446)
-		(stroke
-			(width 0.05)
-			(type solid)
-		)
-		(layer "Edge.Cuts")
-	)
 	(embedded_fonts no)
 )
