File: GACSA EZ-48.kicad_sch (KiCad schematic)
At the start: 49 parts, among them J1 Conn_02x10_Top_Bottom_Mountin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, J2 DIN-5_180degree, J3 Conn_01x10_Socket, J4 Conn_01x10_Socket, Q1 2N4401, U1 6502, U10 74LS244, U2 6520, U3 6520, U4 SN76489, U5 TMS9918A, U6 74LS139, U7 74LS74, U8 7400, U9 74LS244, X1 10.7386MHz

Commit message: Added TMS2732 footprint
Added TMS2732 footprint
Parts:
- removed J1: Conn_02x10_Top_Bottom_MountingPin, Connector_IDC:IDC-Header_2x10-1MP_P2.54mm_Latch6.5mm_Vertical, symbol Connector_Generic_MountingPin:Conn_02x10_Top_Bottom_MountingPin
- added C16, C17, C18, C19, C21, C22, C23, C24, C27, C28, C29, C30, C32, C33, C34, C35, C38, C39, C40, C41, C43, C44, C45, C46: 0.1µF, Capacitor_THT:C_Disc_D7.5mm_W2.5mm_P5.00mm, symbol Device:C
- added C20, C25, C26, C31, C36, C37, C42, C47, C48: 10µF, Capacitor_THT:CP_Radial_D5.0mm_P2.00mm, symbol Device:C_Polarized_Small_US
- added E10, E11, E12, E13, E14, E15, E16, E17, E18, E19, E20, E21, E22, E23, E24, E25, E26, E27, E28, E29, E30, E31, E32, E9: 4116, Package_DIP:DIP-16_W7.62mm_Socket_LongPads, symbol AppleII+:4116
- added J5, J6: Conn_01x10_Socket, Connector_PinSocket_2.54mm:PinSocket_1x10_P2.54mm_Vertical, symbol Connector:Conn_01x10_Socket
- added R8: 75, Resistor_THT:R_Axial_DIN0207_L6.3mm_D2.5mm_P7.62mm_Horizontal, symbol Device:R
- added U11, U12, U13: TMS2732, GACSA EZ-48:TMS 2732, symbol GACSA EZ-48:TMS2732
- added U14, U15: 74LS244, Package_DIP:DIP-20_W7.62mm_LongPads, symbol 74xx:74LS244
- added U16: 74LS138, symbol 74xx:74LS138
- U1, U2, U3: footprint Package_DIP:DIP-40_W15.24mm -> Package_DIP:DIP-40_W15.24mm_LongPads
Connections:
- net +12V: now also C21.1, C22.1, C23.1, C24.1, C25.1, C32.1, C33.1, C34.1, C35.1, C36.1, C43.1, C44.1, C45.1, C46.1, C47.1
- net +12VDC: now also E10.8 (VDD), E11.8 (VDD), E12.8 (VDD), E13.8 (VDD), E14.8 (VDD), E15.8 (VDD), E17.8 (VDD), E18.8 (VDD), E19.8 (VDD), E20.8 (VDD), E21.8 (VDD), E22.8 (VDD), E23.8 (VDD), E25.8 (VDD), E26.8 (VDD), E27.8 (VDD), E28.8 (VDD), E29.8 (VDD), E30.8 (VDD), E31.8 (VDD), E9.8 (VDD)
- net +5V: now also U9.20 (VCC), C26.1, C37.1, C48.1, R8.1
- net +5VDC: now also E10.9 (VCC), E11.9 (VCC), E12.9 (VCC), E13.9 (VCC), E14.9 (VCC), E15.9 (VCC), E17.9 (VCC), E18.9 (VCC), E19.9 (VCC), E20.9 (VCC), E21.9 (VCC), E22.9 (VCC), E23.9 (VCC), E25.9 (VCC), E26.9 (VCC), E27.9 (VCC), E28.9 (VCC), E29.9 (VCC), E30.9 (VCC), E31.9 (VCC), E9.9 (VCC), J5.2 (Pin_2), U11.24 (VCC), U12.24 (VCC), U13.24 (VCC)
- net -5V: now also C16.2, C17.2, C18.2, C19.2, C20.2, C27.2, C28.2, C29.2, C30.2, C31.2, C38.2, C39.2, C40.2, C41.2, C42.2
- net -5VDC: now also E10.1 (VBB), E11.1 (VBB), E12.1 (VBB), E13.1 (VBB), E14.1 (VBB), E15.1 (VBB), E17.1 (VBB), E18.1 (VBB), E19.1 (VBB), E20.1 (VBB), E21.1 (VBB), E22.1 (VBB), E23.1 (VBB), E25.1 (VBB), E26.1 (VBB), E27.1 (VBB), E28.1 (VBB), E29.1 (VBB), E30.1 (VBB), E31.1 (VBB), E9.1 (VBB)
- net A0: now also U11.8 (A0), U12.8 (A0), U13.8 (A0)
- net A1: now also U11.7 (A1), U12.7 (A1), U13.7 (A1)
- net A10: now also U11.19 (A10), U12.19 (A10), U13.19 (A10)
- net A11: now also U11.21 (A11), U12.21 (A11), U13.21 (A11)
- net A2: now also U11.6 (A2), U12.6 (A2), U13.6 (A2)
- net A3: now also U11.5 (A3), U12.5 (A3), U13.5 (A3)
- net A4: now also U11.4 (A4), U12.4 (A4), U13.4 (A4)
- net A5: now also U11.3 (A5), U12.3 (A5), U13.3 (A5)
- net A6: now also U11.2 (A6), U12.2 (A6), U13.2 (A6)
- net A7: now also U11.1 (A7), U12.1 (A7), U13.1 (A7)
- net A8: now also U11.23 (A8), U12.23 (A8), U13.23 (A8)
- net A9: now also U11.22 (A9), U12.22 (A9), U13.22 (A9)
- net ACK: now also J3.10 (Pin_10); no longer J3.9 (Pin_9)
- net D0: now also U11.9 (D0), U12.9 (D0), U13.9 (D0)
- net D1: now also U11.10 (D1), U12.10 (D1), U13.10 (D1)
- net D2: now also U11.11 (D2), U12.11 (D2), U13.11 (D2)
- net D3: now also U11.13 (D3), U12.13 (D3), U13.13 (D3)
- net D4: now also U11.14 (D4), U12.14 (D4), U13.14 (D4)
- net D5: now also U11.15 (D5), U12.15 (D5), U13.15 (D5)
- net D6: now also U11.16 (D6), U12.16 (D6), U13.16 (D6)
- net D7: now also U11.17 (D7), U12.17 (D7), U13.17 (D7)
- net GND: now also C16.1, C17.1, C18.1, C19.1, C20.1, C21.2, C22.2, C23.2, C24.2, C25.2, C26.2, C27.1, C28.1, C29.1, C30.1, C31.1, C32.2, C33.2, C34.2, C35.2, C36.2, C37.2, C38.1, C39.1, C40.1, C41.1, C42.1, C43.2, C44.2, C45.2, C46.2, C47.2, C48.2, E10.16 (GND), E11.16 (GND), E12.16 (GND), E13.16 (GND), E14.16 (GND), E15.16 (GND), E16.16 (GND), E17.16 (GND), E18.16 (GND), E19.16 (GND), E20.16 (GND), E21.16 (GND), E22.16 (GND), E23.16 (GND), E24.16 (GND), E25.16 (GND), E26.16 (GND), E27.16 (GND), E28.16 (GND), E29.16 (GND), E30.16 (GND), E31.16 (GND), E32.16 (GND), E9.16 (GND), J5.1 (Pin_1), U11.12 (GND), U12.12 (GND), U13.12 (GND)
- net PIA0PA0: now also J6.3 (Pin_3)
- net PIA0PA1: now also J6.4 (Pin_4)
- net PIA0PA2: now also J6.5 (Pin_5)
- net PIA0PA3: now also J6.6 (Pin_6)
- net PIA0PA4: now also J6.7 (Pin_7)
- net PIA0PA5: now also J6.8 (Pin_8)
- net PIA0PA6: now also J6.9 (Pin_9)
- net PIA0PB0: now also J5.3 (Pin_3)
- net PIA0PB1: now also J5.4 (Pin_4)
- net PIA0PB2: now also J5.5 (Pin_5)
- net PIA0PB3: now also J5.6 (Pin_6)
- net PIA0PB4: now also J5.7 (Pin_7)
- net PIA0PB5: now also J5.8 (Pin_8)
- net PIA0PB6: now also J5.9 (Pin_9)
- net PIA0PB7: now also J5.10 (Pin_10), J6.10 (Pin_10)
- net VIDOUT: no longer J2.4, Q1.1 (E), R5.1
- net VRAM_ADDR3: now also E12.2 (DI), E20.2 (DI), E28.2 (DI)
- net VRAM_ADDR5: now also E14.2 (DI), E22.2 (DI), E30.2 (DI)
- net VRAM_DATA3: now also E12.14 (D0), E20.14 (D0), E28.14 (D0)
- net VRAM_DATA5: now also E14.14 (D0), E22.14 (D0), E30.14 (D0)
- net at U9.12 (O3a): now also J3.5 (Pin_5); no longer J3.4 (Pin_4)
- net at U9.14 (O2a): now also J3.4 (Pin_4); no longer J3.3 (Pin_3)
- net at U9.16 (O1a): now also J3.3 (Pin_3); no longer J3.2 (Pin_2)
- net at U9.18 (O0a): now also J3.2 (Pin_2); no longer J3.1 (Pin_1)
- net at U9.3 (O3b): now also J3.9 (Pin_9); no longer J3.8 (Pin_8)
- net at U9.5 (O2b): now also J3.8 (Pin_8); no longer J3.7 (Pin_7)
- net at U9.7 (O1b): now also J3.7 (Pin_7); no longer J3.6 (Pin_6)
- net at U9.9 (O0b): now also J3.6 (Pin_6); no longer J3.5 (Pin_5)
- new net STROBE: J3.1 (Pin_1), R8.2
- new net VIDEOOUT: J2.4, Q1.1 (E), R5.1
Other:
- note added: "SYSTEM RAM BANK 0"
- note added: "SYSTEM RAM BANK 1"
- moved on the sheet: C10, C11, C12, C13, C14, C15, C4, C5, C6, C7, C8, C9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

Commit message: Project restarted in a modular way
Project restarted in a modular way
Parts:
- removed C1, C2: 33pF, Capacitor_THT:C_Disc_D7.5mm_W5.0mm_P5.00mm, symbol Device:C
- removed C10, C13, C14, C20, C25, C26, C31, C36, C37, C42, C47, C48: 10µF, Capacitor_THT:CP_Radial_D5.0mm_P2.00mm, symbol Device:C_Polarized_Small_US
- removed C11, C12, C16, C17, C18, C19, C21, C22, C23, C24, C27, C28, C29, C30, C32, C33, C34, C35, C38, C39, C4, C40, C41, C43, C44, C45, C46, C5, C6, C7, C8, C9: 0.1µF, Capacitor_THT:C_Disc_D7.5mm_W2.5mm_P5.00mm, symbol Device:C
- removed C15: 0.1uf, Capacitor_THT:C_Disc_D3.0mm_W1.6mm_P2.50mm, symbol Device:C
- removed C3: 5-50pF, passives:C_Trimmer_THT_5mm, symbol Device:C_Trim_Small
- removed D17: LED, LED_THT:LED_D3.0mm, symbol Device:LED
- removed E1, E10, E11, E12, E13, E14, E15, E16, E17, E18, E19, E2, E20, E21, E22, E23, E24, E25, E26, E27, E28, E29, E3, E30, E31, E32, E4, E5, E6, E7, E8, E9: 4116, Package_DIP:DIP-16_W7.62mm_Socket_LongPads, symbol AppleII+:4116
- removed J2: DIN-5_180degree, symbol Connector:DIN-5_180degree
- removed J3, J4, J5, J6: Conn_01x10_Socket, Connector_PinSocket_2.54mm:PinSocket_1x10_P2.54mm_Vertical, symbol Connector:Conn_01x10_Socket
- removed L1: Ferrite_Bead, Resistor_THT:R_Axial_DIN0207_L6.3mm_D2.5mm_P7.62mm_Horizontal, symbol Device:Ferrite_Bead
- removed Q1: 2N4401, Package_TO_SOT_THT:TO-92L, symbol Device:Q_NPN_EBC
- removed R1, R2: 3.3kΩ, Resistor_THT:R_Axial_DIN0207_L6.3mm_D2.5mm_P10.16mm_Horizontal, symbol Device:R_Small_US
- removed R3: 100Ohm, symbol Device:R_Small_US
- removed R4: 330Ω, Resistor_THT:R_Axial_DIN0207_L6.3mm_D2.5mm_P10.16mm_Horizontal, symbol Device:R_Small_US
- removed R5, R8: 75, Resistor_THT:R_Axial_DIN0207_L6.3mm_D2.5mm_P7.62mm_Horizontal, symbol Device:R
- removed R6: R_Variable, Resistor_THT:R_Axial_DIN0207_L6.3mm_D2.5mm_P10.16mm_Horizontal, symbol Device:R_Variable
- removed R7: 470, Resistor_THT:R_Axial_DIN0207_L6.3mm_D2.5mm_P7.62mm_Horizontal, symbol Device:R
- removed U10, U14, U15, U9: 74LS244, Package_DIP:DIP-20_W7.62mm_LongPads, symbol 74xx:74LS244
- removed U11, U12, U13: TMS2732, GACSA EZ-48:TMS 2732, symbol GACSA EZ-48:TMS2732
- removed U16: 74LS138, symbol 74xx:74LS138
- removed U2, U3: 6520, Package_DIP:DIP-40_W15.24mm_LongPads, symbol Interface:6821
- removed U4: SN76489, Package_DIP:DIP-16_W7.62mm_Socket_LongPads, symbol LeakoChips:SN76489AN
- removed U5: TMS9918A, Package_DIP:DIP-40_W15.24mm_Socket_LongPads, symbol LeakoChips:TMS9918A
- removed U6: 74LS139, Package_DIP:DIP-16_W7.62mm_LongPads, symbol 74xx:74LS139
- removed U7: 74LS74, symbol 74xx:74LS74
- removed U8: 7400, symbol 74xx:7400
- removed X1: 10.7386MHz, Crystal:Crystal_HC49-4H_Vertical, symbol Device:Crystal_GND3_Small
- added IC1: TMS9918A, Package_DIP:DIP-40_W15.24mm_Socket, symbol yamaha:TMS9918A
- added R1: 1000 Ohm, Resistor_THT:R_Axial_DIN0204_L3.6mm_D1.6mm_P7.62mm_Horizontal, symbol Device:R_US
- added RA1: 1000 Ohm, Resistor_THT:R_Array_SIP8, symbol Device:R_Network07_US
- added U1: 74LS00, symbol 74xx:74LS00
- added U3: 74LS139, Package_DIP:DIP-16_W7.62mm_LongPads, symbol 74xx:74LS139
- added U4, U6: 74LS138, Package_DIP:DIP-16_W7.62mm_LongPads, symbol 74xx:74LS138
- added U5: 74LS00, Package_DIP:DIP-14_W7.62mm_LongPads, symbol 74xx:74LS00
- added Y1: 1.79 Mhz, Oscillator:Oscillator_DIP-8_LargePads, symbol Oscillator:CXO_DIP8
- CP1: footprint Connector_IDC:IDC-Header_2x03_P2.54mm_Vertical -> Connector_Harwin:Harwin_LTek-Male_2x03_P2.00mm_Vertical
- U2: renamed from U1; footprint Package_DIP:DIP-40_W15.24mm_LongPads -> Package_DIP:DIP-40_W15.24mm_Socket_LongPads
Connections:
- net +5VDC is gone; now on net +5V: U2.8 (VCC)
- net +5V: now also R1.1, RA1.1 (common), U1.14 (VCC), U3.16 (VCC), U4.16 (VCC), U5.14 (VCC), U6.16 (VCC), Y1.8 (Vcc)
- net A10: now also U6.3 (A2)
- net A11: now also U1.13, U5.1, U5.2
- net A12: now also U3.14 (A0)
- net A13: now also U3.13 (A1)
- net A14: now also U3.2 (A0)
- net A15: now also U3.3 (A1)
- net A4: now also U4.1 (A0)
- net A5: now also U4.2 (A1)
- net A6: now also U4.3 (A2)
- net A7: now also U4.6 (E3)
- net A8: now also U6.1 (A0)
- net A9: now also U6.2 (A1)
- net GND: now also U1.7 (GND), U3.1 (E), U3.8 (GND), U4.8 (GND), U5.7 (GND), U6.8 (GND), Y1.4 (GND); no longer U2.38 (~{SO})
- net PHI1: now also U4.5 (E2); no longer U2.3 (ϕ1)
- net PHI2: now also U1.1, U1.10
- net ~{READ}: now also U1.3
- net ~{RESET}: now also RA1.3 (R2)
- net ~{WRITE}: now also U1.8
- net 1.79Mhz: no longer names the net of U2.37 (ϕ0)
- net R/~{W} renamed ~{R}/W
- net ~{R}/W: now also U1.2, U1.4, U1.5
- net ~{CPUIRQ}: no longer names the net of U2.4 (~{IRQ})
- net ~{CPUNMI}: no longer names the net of U2.6 (~{NMI})
- new net: U1.6, U1.9
- new net: U5.3, U5.4
- new net: U5.6, U6.4 (E1), U6.5 (E2)
- new net: R1.2, U6.6 (E3)
- new net: U3.15 (E), U3.7 (O3)
- new net ~{C000-C0FF}: U4.4 (E1), U6.15 (O0)
- new net ~{CARDROM}: U1.11
- new net ~{DEVSEL0}: U4.15 (O0)
- new net ~{DEVSEL1}: U4.14 (O1)
- new net ~{DEVSEL2}: U4.13 (O2)
- new net ~{DEVSEL3}: U4.12 (O3)
- new net ~{DEVSEL4}: U4.11 (O4)
- new net ~{DEVSEL5}: U4.10 (O5)
- new net ~{DEVSEL6}: U4.9 (O6)
- new net ~{DEVSEL7}: U4.7 (O7)
- new net ~{DMA}: RA1.5 (R4)
- new net ~{IOROM1}: U6.14 (O1)
- new net ~{IOROM2}: U6.13 (O2)
- new net ~{IOROM3}: U6.12 (O3)
- new net ~{IOROM4}: U6.11 (O4)
- new net ~{IOROM5}: U6.10 (O5)
- new net ~{IOROM6}: U6.9 (O6)
- new net ~{IOROM7}: U6.7 (O7)
- new net ~{IOSEL}: U1.12, U3.12 (O0), U5.5
- new net ~{NMI}: RA1.2 (R1)
- new net ~{RAMSEL0}: U3.4 (O0)
- new net ~{RAMSEL1}: U3.5 (O1)
- new net ~{RAMSEL2}: U3.6 (O2)
- new net ~{RDY}: RA1.4 (R3)
- new net ~{ROMSEL0}: U3.11 (O1)
- new net ~{ROMSEL1}: U3.10 (O2)
- new net ~{ROMSEL2}: U3.9 (O3)
- no-connect marks 5 -> 10
Other:
- note added: "$0000-$3FFF 16K $4000-$7FFF 16K $8000-$BFFF 16K"
- note added: "$C000-$CFFF I/O $D000-$DFFF 4K $E000-$EFFF 4K $F000-$FFFF 4K"
- note added: "256 Bytes ROM for each expansion card"
- note added: "2K ROM at $C800-$CFFF *TODO*: Implement a scheme to strobe it on each expansion card"
- note added: "C080-C08F C090-C09F C0A0-C0AF C0B0-C0BF C0C0-C0CF C0D0-C0DF C0E0-C0EF C0F0-C0FF"
- note added: "C100-C1FF C200-C2FF C300-C3FF C400-C4FF C500-C5FF C600-C6FF C700-C7FF"
- note added: "TMS9918 GPU 6520 PIA (Keyboard, Joystick, Tape) 6520 PIA (Sound, Printer) TMS5200 Speech Synth (unpopulated) 6551 RS232 Card (unpopulated) Expansion slot Expansion slot Expansion slot"
- note added: "~{C000-C0FF} are I/O ports' Device Selectors"
- note added: "~{C000-C7FF}"
- note removed: "0-200Ohm"
- note removed: "Keyboard Connector"
- note removed: "PARALLEL PORT"
- note removed: "READ/WRITE LOGIC"
- note removed: "SYSTEM RAM BANK 0"
- note removed: "SYSTEM RAM BANK 1"
- note removed: "VIDEO RAM"
- company: (none) -> Original (R) 1979, 1981 Grupo Atlacatl Comercial S.A.
- title: (none) -> GACSA EZ-48 Computer Schematic Replica
- moved on the sheet: CP1, U2

Commit message: Checked on Schematic Documentation
Checked on Schematic Documentation
Parts:
- removed IC1: TMS9918A, Package_DIP:DIP-40_W15.24mm_Socket, symbol yamaha:TMS9918A
- removed unit 3 of U1
- removed unit 4 of U5
- removed unit 3 of U5
- removed Y1: 1.79 Mhz, Oscillator:Oscillator_DIP-8_LargePads, symbol Oscillator:CXO_DIP8
- added C1, C10, C2, C3, C4, C5, C6, C7, C8, C9: 47uF, Capacitor_THT:C_Disc_D7.5mm_W2.5mm_P5.00mm, symbol Device:C
- added C29: .1uf, Capacitor_THT:C_Rect_L7.0mm_W2.0mm_P5.00mm, symbol Device:C
- added C30: 10uf, Capacitor_THT:CP_Radial_D4.0mm_P2.00mm, symbol Device:C
- added D1: LED, LED_THT:LED_D3.0mm, symbol Device:LED
- added R1: 330Ω, Resistor_THT:R_Axial_DIN0207_L6.3mm_D2.5mm_P10.16mm_Horizontal, symbol Device:R_Small_US
- added R11: 220k, Resistor_THT:R_Axial_DIN0207_L6.3mm_D2.5mm_P7.62mm_Horizontal, symbol Device:R
- added R12: 150K, Resistor_THT:R_Axial_DIN0207_L6.3mm_D2.5mm_P7.62mm_Horizontal, symbol Device:R
- added R13: 1K, Resistor_THT:R_Axial_DIN0207_L6.3mm_D2.5mm_P7.62mm_Horizontal, symbol Device:R
- added R14, R15: 2200 Ohm, symbol Device:R
- added R2: 470 Ω, Resistor_THT:R_Axial_DIN0204_L3.6mm_D1.6mm_P7.62mm_Horizontal, symbol Device:R_US
- added U11, U6, U9: TMS2732, Package_DIP:DIP-24_18.0mmx34.29mm_W15.24mm_Socket_LongPads, symbol GACSA EZ-48:TMS2732
- added U12: 74LS00, symbol 74xx:74LS00
- added unit 3 of U2
- added U25: TI555, Package_DIP:DIP-8_W7.62mm_Socket_LongPads, symbol Timer:LM555xN
- added U4: TMS6064, Package_DIP:DIP-28_W15.24mm_Socket_LongPads, symbol Memory_RAM:HY6264AxP
- added U8: 74LS74, symbol 74xx:74LS74
- R3: renamed from R1; value 1000 Ohm -> 1000 Ω
- RA1: value 1000 Ohm -> 1000Ω
- U5: footprint Package_DIP:DIP-14_W7.62mm_LongPads -> Package_DIP:DIP-14_W7.62mm_Socket_LongPads
- U5: renamed from U1; footprint (none) -> Package_DIP:DIP-14_W7.62mm_Socket_LongPads
- renumbered U2 to U1, U6 to U10, U1 to U2, U5 to U2, U4 to U7
Connections:
- net ~{RDY} is gone; now on net ~{DMA}: RA1.4 (R3)
- net +5V: now also C1.2, C10.2, C2.2, C3.2, C4.2, C5.2, C6.2, C7.2, C8.2, C9.2, D1.2 (A), R11.1, R14.1, R15.2, R2.2, U11.24 (VCC), U12.14 (VCC), U25.4 (R), U25.8 (VCC), U4.28 (VCC), U6.24 (VCC), U8.1 (~{R}), U8.14 (VCC), U8.4 (~{S}), U9.24 (VCC)
- net A0: now also U11.8 (A0), U4.10 (A0), U6.8 (A0), U9.8 (A0)
- net A1: now also U11.7 (A1), U4.9 (A1), U6.7 (A1), U9.7 (A1)
- net A10: now also U11.19 (A10), U4.21 (A10), U6.19 (A10), U9.19 (A10)
- net A11: now also U2.12, U2.13, U5.5, U11.21 (A11), U4.23 (A11), U6.21 (A11), U9.21 (A11); no longer U2.1, U2.2, U5.13
- net A12: now also U4.2 (A12)
- net A2: now also U11.6 (A2), U4.8 (A2), U6.6 (A2), U9.6 (A2)
- net A3: now also U11.5 (A3), U4.7 (A3), U6.5 (A3), U9.5 (A3)
- net A4: now also U11.4 (A4), U4.6 (A4), U6.4 (A4), U9.4 (A4)
- net A5: now also U11.3 (A5), U4.5 (A5), U6.3 (A5), U9.3 (A5)
- net A6: now also U11.2 (A6), U4.4 (A6), U6.2 (A6), U9.2 (A6)
- net A7: now also U11.1 (A7), U4.3 (A7), U6.1 (A7), U9.1 (A7)
- net A8: now also U11.23 (A8), U4.25 (A8), U6.23 (A8), U9.23 (A8)
- net A9: now also U11.22 (A9), U4.24 (A9), U6.22 (A9), U9.22 (A9)
- net D0: now also U11.9 (D0), U4.11 (I/O0), U6.9 (D0), U9.9 (D0)
- net D1: now also U11.10 (D1), U4.12 (I/O1), U6.10 (D1), U9.10 (D1)
- net D2: now also U11.11 (D2), U4.13 (I/O2), U6.11 (D2), U9.11 (D2)
- net D3: now also U11.13 (D3), U4.15 (I/O3), U6.13 (D3), U9.13 (D3)
- net D4: now also U11.14 (D4), U4.16 (I/O4), U6.14 (D4), U9.14 (D4)
- net D5: now also U11.15 (D5), U4.17 (I/O5), U6.15 (D5), U9.15 (D5)
- net D6: now also U11.16 (D6), U4.18 (I/O6), U6.16 (D6), U9.16 (D6)
- net D7: now also U11.17 (D7), U4.19 (I/O7), U6.17 (D7), U9.17 (D7)
- net GND: now also C1.1, C10.1, C2.1, C29.2, C3.1, C30.2, C4.1, C5.1, C6.1, C7.1, C8.1, C9.1, R1.2, R12.1, R13.2, U11.12 (GND), U12.7 (GND), U25.1 (GND), U4.14 (GND), U6.12 (GND), U8.7 (GND), U9.12 (GND)
- net PHI1: now also U1.3 (ϕ1)
- net PHI2: now also U2.10
- net ~{CARDROM}: now also U5.6; no longer U5.11
- net ~{DMA}: no longer RA1.5 (R4)
- net ~{IOSEL}: now also U5.2, U5.4; no longer U5.12, U5.5
- net ~{NMI}: now also U1.6 (~{NMI}), R15.1
- net ~{RAMSEL0}: now also U4.20 (~{CS1})
- net ~{READ}: now also U11.20 (~{G}/VPRG), U4.22 (~{OE}), U6.20 (~{G}/VPRG), U9.20 (~{G}/VPRG)
- net ~{RESET}: now also R13.1, U12.6
- net ~{ROMSEL0}: now also U6.18 (~{E})
- net ~{ROMSEL1}: now also U9.18 (~{E})
- net ~{ROMSEL2}: now also U11.18 (~{E})
- net ~{WRITE}: now also U2.8, U4.27 (~{WE})
- net at U2.6: now also U2.9
- net at U10.4 (E1), U10.5 (E2): now also U5.3; no longer U5.6
- net 1.79Mhz: now reaches U1.37 (ϕ0)
- net 1.79Mhz: now also U8.5 (Q)
- net ~{IRQ}: now reaches U1.4 (~{IRQ})
- net ~{IRQ}: now also RA1.5 (R4), R14.2
- new net: D1.1 (K), R1.1
- new net: C29.1, R11.2, U25.2 (TR)
- new net: U12.4, U12.5, U25.3 (Q)
- new net: C30.1, R12.2, U25.6 (THR), U25.7 (DIS)
- new net: U2.11, U5.1
- new net: R2.1, U4.26 (CS2)
- new net: U8.2 (D), U8.6 (~{Q})
- new net 3.58MHz: U8.3 (C)
- no-connect marks 10 -> 16
Other:
- added sheet Dynamic RAM (dram.kicad_sch)
- added sheet Expansion Slots (slots.kicad_sch)
- added sheet Peripherals and Sound (pia.kicad_sch)
- added sheet Video Interface (video.kicad_sch)
- note added: "RESET CIRCUIT"
- note added: "Unpopulated SRAM on EZ-48 board"
- moved on the sheet: CP1
